File: keyboard/matrix.kicad_sch (KiCad schematic)
At the start: 134 parts, among them SW10 8, SW11 9, SW12 0, SW13 -_, SW14 +=, SW15 BSPC, SW16 DEL, SW17 TAB, SW18 Q, SW19 W, SW2 ESC, SW20 E, SW21 R, SW22 T, SW23 Y, SW24 U, SW25 I, SW26 O, SW27 P, SW28 {[, SW29 }], SW3 1, SW30 |\, SW31 PGUP, SW32 CAPS, SW33 A, SW34 S, SW35 D, SW36 F, SW37 G, SW38 H, SW39 J, SW4 2, SW40 K, SW41 L, SW42 :;, SW43 "', SW44 ENTER, SW45 PGDN, SW46 SHIFT, SW47 Z, SW48 X, SW49 C, SW5 3, SW50 V, SW51 B, SW52 N, SW53 M, SW54 <,, SW55 >., SW56 ?/, SW57 SHIFT, SW58 UP, SW59 END, SW6 4, SW60 CTRL, SW61 WIN, SW62 ALT, SW63 SPACE, SW64 FN, SW65 CTRL, SW66 LEFT, SW67 DOWN, SW68 RIGHT, SW7 5, SW8 6, SW9 7

Commit message: Assigned footprints + fixed errors
Parts:
- D1, D10, D11, D12, D13, D14, D15, D16, D17, D18, D19, D2, D20, D21, D22, D23, D24, D25, D26, D27, D28, D29, D3, D30, D31, D32, D33, D34, D35, D36, D37, D38, D39, D4, D40, D41, D42, D43, D44, D45, D46, D47, D48, D49, D5, D50, D51, D52, D53, D54, D55, D56, D57, D58, D59, D6, D60, D61, D62, D63, D64, D65, D66, D67, D7, D8, D9: footprint (none) -> Diode_SMD:D_SOD-123
- SW10, SW11, SW12, SW13, SW14, SW16, SW18, SW19, SW2, SW20, SW21, SW22, SW23, SW24, SW25, SW26, SW27, SW28, SW29, SW3, SW31, SW33, SW34, SW35, SW36, SW37, SW38, SW39, SW4, SW40, SW41, SW42, SW43, SW44, SW45, SW47, SW48, SW49, SW5, SW50, SW51, SW52, SW53, SW54, SW55, SW56, SW58, SW59, SW6, SW66, SW67, SW68, SW7, SW8, SW9: footprint (none) -> Button_Switch_Keyboard:SW_Cherry_MX_1.00u_PCB
- SW15: footprint (none) -> Button_Switch_Keyboard:SW_Cherry_MX_2.00u_PCB
- SW17, SW30, SW60: footprint (none) -> Button_Switch_Keyboard:SW_Cherry_MX_1.50u_PCB
- SW32, SW57: footprint (none) -> Button_Switch_Keyboard:SW_Cherry_MX_1.75u_PCB
- SW46: footprint (none) -> Button_Switch_Keyboard:SW_Cherry_MX_2.25u_PCB
- SW61, SW64, SW65: footprint (none) -> Button_Switch_Keyboard:SW_Cherry_MX_1.25u_PCB
- SW62: footprint (none) -> Button_Switch_Keyboard:SW_Cherry_MX_1.50_PCB
- SW63: footprint (none) -> Button_Switch_Keyboard:SW_Cherry_MX_6.50u_PCB
Connections:
- net col0: no longer D1.1 (K), D10.1 (K), D11.1 (K), D12.1 (K), D13.1 (K), D14.1 (K), D15.1 (K), D16.1 (K), D17.1 (K), D18.1 (K), D19.1 (K), D2.1 (K), D20.1 (K), D21.1 (K), D22.1 (K), D23.1 (K), D24.1 (K), D25.1 (K), D26.1 (K), D27.1 (K), D28.1 (K), D29.1 (K), D3.1 (K), D30.1 (K), D31.1 (K), D32.1 (K), D33.1 (K), D34.1 (K), D35.1 (K), D36.1 (K), D37.1 (K), D38.1 (K), D39.1 (K), D4.1 (K), D40.1 (K), D41.1 (K), D42.1 (K), D43.1 (K), D44.1 (K), D45.1 (K), D46.1 (K), D47.1 (K), D48.1 (K), D49.1 (K), D5.1 (K), D50.1 (K), D51.1 (K), D52.1 (K), D53.1 (K), D54.1 (K), D55.1 (K), D56.1 (K), D57.1 (K), D58.1 (K), D59.1 (K), D6.1 (K), D60.1 (K), D61.1 (K), D62.1 (K), D63.1 (K), D64.1 (K), D65.1 (K), D66.1 (K), D67.1 (K), D7.1 (K), D8.1 (K), D9.1 (K), SW10.2, SW11.2, SW12.2, SW13.2, SW14.2, SW15.2, SW16.2, SW18.2, SW19.2, SW20.2, SW21.2, SW22.2, SW23.2, SW24.2, SW25.2, SW26.2, SW27.2, SW28.2, SW29.2, SW3.2, SW30.2, SW31.2, SW33.2, SW34.2, SW35.2, SW36.2, SW37.2, SW38.2, SW39.2, SW4.2, SW40.2, SW41.2, SW42.2, SW43.2, SW44.2, SW45.2, SW47.2, SW48.2, SW49.2, SW5.2, SW50.2, SW51.2, SW52.2, SW53.2, SW54.2, SW55.2, SW56.2, SW57.2, SW58.2, SW59.2, SW6.2, SW61.2, SW62.2, SW63.2, SW64.2, SW65.2, SW66.2, SW67.2, SW68.2, SW7.2, SW8.2, SW9.2
- new net col1: SW18.2, SW3.2, SW33.2, SW47.2, SW61.2
- new net col10: SW12.2, SW27.2, SW42.2, SW56.2, SW64.2
- new net col11: SW13.2, SW28.2, SW43.2, SW65.2
- new net col12: SW14.2, SW29.2, SW57.2, SW66.2
- new net col13: SW15.2, SW30.2, SW44.2, SW58.2, SW67.2
- new net col14: SW16.2, SW31.2, SW45.2, SW59.2, SW68.2
- new net col2: SW19.2, SW34.2, SW4.2, SW48.2, SW62.2
- new net col3: SW20.2, SW35.2, SW49.2, SW5.2
- new net col4: SW21.2, SW36.2, SW50.2, SW6.2
- new net col5: SW22.2, SW37.2, SW51.2, SW7.2
- new net col6: SW23.2, SW38.2, SW52.2, SW63.2, SW8.2
- new net col7: SW24.2, SW39.2, SW53.2, SW9.2
- new net col8: SW10.2, SW25.2, SW40.2, SW54.2
- new net col9: SW11.2, SW26.2, SW41.2, SW55.2
- new net row0: D1.1 (K), D10.1 (K), D11.1 (K), D12.1 (K), D13.1 (K), D14.1 (K), D15.1 (K), D2.1 (K), D3.1 (K), D4.1 (K), D5.1 (K), D6.1 (K), D7.1 (K), D8.1 (K), D9.1 (K)
- new net row1: D16.1 (K), D17.1 (K), D18.1 (K), D19.1 (K), D20.1 (K), D21.1 (K), D22.1 (K), D23.1 (K), D24.1 (K), D25.1 (K), D26.1 (K), D27.1 (K), D28.1 (K), D29.1 (K), D30.1 (K)
- new net row2: D31.1 (K), D32.1 (K), D33.1 (K), D34.1 (K), D35.1 (K), D36.1 (K), D37.1 (K), D38.1 (K), D39.1 (K), D40.1 (K), D41.1 (K), D42.1 (K), D43.1 (K), D44.1 (K)
- new net row3: D45.1 (K), D46.1 (K), D47.1 (K), D48.1 (K), D49.1 (K), D50.1 (K), D51.1 (K), D52.1 (K), D53.1 (K), D54.1 (K), D55.1 (K), D56.1 (K), D57.1 (K), D58.1 (K)
- new net row4: D59.1 (K), D60.1 (K), D61.1 (K), D62.1 (K), D63.1 (K), D64.1 (K), D65.1 (K), D66.1 (K), D67.1 (K)

Commit message: Finished keyboard switch layout for PCB
Parts:
- SW10, SW11, SW12, SW13, SW14, SW16, SW18, SW19, SW2, SW20, SW21, SW22, SW23, SW24, SW25, SW26, SW27, SW28, SW29, SW3, SW31, SW33, SW34, SW35, SW36, SW37, SW38, SW39, SW4, SW40, SW41, SW42, SW43, SW45, SW47, SW48, SW49, SW5, SW50, SW51, SW52, SW53, SW54, SW55, SW56, SW58, SW59, SW6, SW66, SW67, SW68, SW7, SW8, SW9: footprint Button_Switch_Keyboard:SW_Cherry_MX_1.00u_PCB -> MX:MXOnly-1U
- SW15: footprint Button_Switch_Keyboard:SW_Cherry_MX_2.00u_PCB -> MX:MXOnly-2U
- SW17, SW30, SW60: footprint Button_Switch_Keyboard:SW_Cherry_MX_1.50u_PCB -> MX:MXOnly-1.5U
- SW32, SW57: footprint Button_Switch_Keyboard:SW_Cherry_MX_1.75u_PCB -> MX:MXOnly-1.75U
- SW44: footprint Button_Switch_Keyboard:SW_Cherry_MX_1.00u_PCB -> MX:MXOnly-2.25U
- SW46: footprint Button_Switch_Keyboard:SW_Cherry_MX_2.25u_PCB -> MX:MXOnly-2.25U
- SW61, SW64, SW65: footprint Button_Switch_Keyboard:SW_Cherry_MX_1.25u_PCB -> MX:MXOnly-1.25U
- SW62: footprint Button_Switch_Keyboard:SW_Cherry_MX_1.50_PCB -> MX:MXOnly-1.5U
- SW63: footprint Button_Switch_Keyboard:SW_Cherry_MX_6.50u_PCB -> MX:MXOnly-6.25U

Commit message: Finished diode layout and changed switch footprints to no-LED
Parts:
- SW10, SW11, SW12, SW13, SW14, SW16, SW18, SW19, SW2, SW20, SW21, SW22, SW23, SW24, SW25, SW26, SW27, SW28, SW29, SW3, SW31, SW33, SW34, SW35, SW36, SW37, SW38, SW39, SW4, SW40, SW41, SW42, SW43, SW45, SW47, SW48, SW49, SW5, SW50, SW51, SW52, SW53, SW54, SW55, SW56, SW58, SW59, SW6, SW66, SW67, SW68, SW7, SW8, SW9: footprint MX:MXOnly-1U -> MX:MXOnly-1U-NoLED
- SW15: footprint MX:MXOnly-2U -> MX:MXOnly-2U-NoLED
- SW17, SW30, SW60, SW62: footprint MX:MXOnly-1.5U -> MX:MXOnly-1.5U-NoLED
- SW32, SW57: footprint MX:MXOnly-1.75U -> MX:MXOnly-1.75U-NoLED
- SW44, SW46: footprint MX:MXOnly-2.25U -> MX:MXOnly-2.25U-NoLED
- SW61, SW64, SW65: footprint MX:MXOnly-1.25U -> MX:MXOnly-1.25U-NoLED
- SW63: footprint MX:MXOnly-6.25U -> MX:MXOnly-6.25U-ReversedStabilizers-NoLED
Changed lines of the file:
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@@
 			)
 		)
-		(property "Footprint" "MX:MXOnly-1U"
+		(property "Footprint" "MX:MXOnly-1U-NoLED"
 			(at 250.19 114.3 0)
 			(effects
@@
 			)
 		)
-		(property "Footprint" "MX:MXOnly-1.75U"
+		(property "Footprint" "MX:MXOnly-1.75U-NoLED"
 			(at 55.88 139.7 0)
 			(effects
@@
 			)
 		)
-		(property "Footprint" "MX:MXOnly-1.5U"
+		(property "Footprint" "MX:MXOnly-1.5U-NoLED"
 			(at 55.88 190.5 0)
 			(effects
@@
 			)
 		)
-		(property "Footprint" "MX:MXOnly-1U"
+		(property "Footprint" "MX:MXOnly-1U-NoLED"
 			(at 99.06 114.3 0)
 			(effects
@@
 			)
 		)
-		(property "Footprint" "MX:MXOnly-1U"
+		(property "Footprint" "MX:MXOnly-1U-NoLED"
 			(at 99.06 139.7 0)
 			(effects
@@
 			)
 		)
-		(property "Footprint" "MX:MXOnly-1U"
+		(property "Footprint" "MX:MXOnly-1U-NoLED"
 			(at 293.37 139.7 0)
 			(effects
@@
 			)
 		)
-		(property "Footprint" "MX:MXOnly-1.5U"
+		(property "Footprint" "MX:MXOnly-1.5U-NoLED"
 			(at 99.06 190.5 0)
 			(effects
@@
 			)
 		)
-		(property "Footprint" "MX:MXOnly-1U"
+		(property "Footprint" "MX:MXOnly-1U-NoLED"
 			(at 228.6 114.3 0)
 			(effects
@@
 			)
 		)
-		(property "Footprint" "MX:MXOnly-1U"
+		(property "Footprint" "MX:MXOnly-1U-NoLED"
 			(at 250.19 139.7 0)
 			(effects
@@
 			)
 		)
-		(property "Footprint" "MX:MXOnly-1U"
+		(property "Footprint" "MX:MXOnly-1U-NoLED"
 			(at 120.65 114.3 0)
 			(effects
@@
 			)
 		)
-		(property "Footprint" "MX:MXOnly-1U"
+		(property "Footprint" "MX:MXOnly-1U-NoLED"
 			(at 142.24 88.9 0)
 			(effects
@@
 			)
 		)
-		(property "Footprint" "MX:MXOnly-1U"
+		(property "Footprint" "MX:MXOnly-1U-NoLED"
 			(at 185.42 165.1 0)
 			(effects
@@
 			)
 		)
-		(property "Footprint" "MX:MXOnly-1U"
+		(property "Footprint" "MX:MXOnly-1U-NoLED"
 			(at 228.6 165.1 0)
 			(effects
@@
 			)
 		)
-		(property "Footprint" "MX:MXOnly-1U"
+		(property "Footprint" "MX:MXOnly-1U-NoLED"
 			(at 142.24 165.1 0)
 			(effects
@@
 			)
 		)
-		(property "Footprint" "MX:MXOnly-1U"
+		(property "Footprint" "MX:MXOnly-1U-NoLED"
 			(at 55.88 88.9 0)
 			(effects
@@
 			)
 		)
-		(property "Footprint" "MX:MXOnly-2.25U"
+		(property "Footprint" "MX:MXOnly-2.25U-NoLED"
 			(at 336.55 139.7 0)
 			(effects
@@
 			)
 		)
-		(property "Footprint" "MX:MXOnly-1U"
+		(property "Footprint" "MX:MXOnly-1U-NoLED"
 			(at 314.96 88.9 0)
 			(effects
@@
 			)
 		)
-		(property "Footprint" "MX:MXOnly-1.5U"
+		(property "Footprint" "MX:MXOnly-1.5U-NoLED"
 			(at 336.55 114.3 0)
 			(effects
@@
 			)
 		)
-		(property "Footprint" "MX:MXOnly-1U"
+		(property "Footprint" "MX:MXOnly-1U-NoLED"
 			(at 293.37 88.9 0)
 			(effects
@@
 			)
 		)
-		(property "Footprint" "MX:MXOnly-1U"
+		(property "Footprint" "MX:MXOnly-1U-NoLED"
 			(at 142.24 114.3 0)
 			(effects
@@
 			)
 		)
-		(property "Footprint" "MX:MXOnly-1U"
+		(property "Footprint" "MX:MXOnly-1U-NoLED"
 			(at 358.14 88.9 0)
 			(effects
@@
 			)
 		)
-		(property "Footprint" "MX:MXOnly-1U"
+		(property "Footprint" "MX:MXOnly-1U-NoLED"
 			(at 271.78 114.3 0)
 			(effects
@@
 			)
 		)
-		(property "Footprint" "MX:MXOnly-1U"
+		(property "Footprint" "MX:MXOnly-1U-NoLED"
 			(at 207.01 114.3 0)
 			(effects
@@
 			)
 		)
-		(property "Footprint" "MX:MXOnly-1U"
+		(property "Footprint" "MX:MXOnly-1U-NoLED"
 			(at 120.65 165.1 0)
 			(effects
@@
 			)
 		)
-		(property "Footprint" "MX:MXOnly-1U"
+		(property "Footprint" "MX:MXOnly-1U-NoLED"
 			(at 185.42 139.7 0)
 			(effects
@@
 			)
 		)
-		(property "Footprint" "MX:MXOnly-6.25U"
+		(property "Footprint" "MX:MXOnly-6.25U-ReversedStabilizers-NoLED"
 			(at 185.42 190.5 0)
 			(effects
@@
 			)
 		)
-		(property "Footprint" "MX:MXOnly-1U"
+		(property "Footprint" "MX:MXOnly-1U-NoLED"
 			(at 77.47 114.3 0)
 			(effects
@@
 			)
 		)
-		(property "Footprint" "MX:MXOnly-1U"
+		(property "Footprint" "MX:MXOnly-1U-NoLED"
 			(at 77.47 139.7 0)
 			(effects
@@
 			)
 		)
-		(property "Footprint" "MX:MXOnly-1U"
+		(property "Footprint" "MX:MXOnly-1U-NoLED"
 			(at 228.6 139.7 0)
 			(effects
@@
 			)
 		)
-		(property "Footprint" "MX:MXOnly-1U"
+		(property "Footprint" "MX:MXOnly-1U-NoLED"
 			(at 336.55 165.1 0)
 			(effects
@@
 			)
 		)
-		(property "Footprint" "MX:MXOnly-1U"
+		(property "Footprint" "MX:MXOnly-1U-NoLED"
 			(at 120.65 139.7 0)
 			(effects
@@
 			)
 		)
-		(property "Footprint" "MX:MXOnly-2.25U"
+		(property "Footprint" "MX:MXOnly-2.25U-NoLED"
 			(at 55.88 165.1 0)
 			(effects
@@
 			)
 		)
-		(property "Footprint" "MX:MXOnly-1U"
+		(property "Footprint" "MX:MXOnly-1U-NoLED"
 			(at 163.83 88.9 0)
 			(effects
@@
 			)
 		)
-		(property "Footprint" "MX:MXOnly-1U"
+		(property "Footprint" "MX:MXOnly-1U-NoLED"
 			(at 142.24 139.7 0)
 			(effects
@@
 			)
 		)
-		(property "Footprint" "MX:MXOnly-1U"
+		(property "Footprint" "MX:MXOnly-1U-NoLED"
 			(at 163.83 114.3 0)
 			(effects
@@
 			)
 		)
-		(property "Footprint" "MX:MXOnly-1U"
+		(property "Footprint" "MX:MXOnly-1U-NoLED"
 			(at 271.78 88.9 0)
 			(effects
@@
 			)
 		)
-		(property "Footprint" "MX:MXOnly-1U"
+		(property "Footprint" "MX:MXOnly-1U-NoLED"
 			(at 358.14 139.7 0)
 			(effects
@@
 			)
 		)
-		(property "Footprint" "MX:MXOnly-1U"
+		(property "Footprint" "MX:MXOnly-1U-NoLED"
 			(at 250.19 165.1 0)
 			(effects
@@
 			)
 		)
-		(property "Footprint" "MX:MXOnly-1U"
+		(property "Footprint" "MX:MXOnly-1U-NoLED"
 			(at 99.06 88.9 0)
 			(effects
@@
 			)
 		)
-		(property "Footprint" "MX:MXOnly-1U"
+		(property "Footprint" "MX:MXOnly-1U-NoLED"
 			(at 314.96 190.5 0)
 			(effects
@@
 			)
 		)
-		(property "Footprint" "MX:MXOnly-1U"
+		(property "Footprint" "MX:MXOnly-1U-NoLED"
 			(at 271.78 165.1 0)
 			(effects
@@
 			)
 		)
-		(property "Footprint" "MX:MXOnly-1U"
+		(property "Footprint" "MX:MXOnly-1U-NoLED"
 			(at 314.96 114.3 0)
 			(effects
@@
 			)
 		)
-		(property "Footprint" "MX:MXOnly-1U"
+		(property "Footprint" "MX:MXOnly-1U-NoLED"
 			(at 207.01 88.9 0)
 			(effects
@@
 			)
 		)
-		(property "Footprint" "MX:MXOnly-1U"
+		(property "Footprint" "MX:MXOnly-1U-NoLED"
 			(at 358.14 114.3 0)
 			(effects
@@
 			)
 		)
-		(property "Footprint" "MX:MXOnly-1U"
+		(property "Footprint" "MX:MXOnly-1U-NoLED"
 			(at 250.19 88.9 0)
 			(effects
@@
 			)
 		)
-		(property "Footprint" "MX:MXOnly-1U"
+		(property "Footprint" "MX:MXOnly-1U-NoLED"
 			(at 271.78 139.7 0)
 			(effects
@@
 			)
 		)
-		(property "Footprint" "MX:MXOnly-1U"
+		(property "Footprint" "MX:MXOnly-1U-NoLED"
 			(at 185.42 114.3 0)
 			(effects
@@
 			)
 		)
-		(property "Footprint" "MX:MXOnly-1U"
+		(property "Footprint" "MX:MXOnly-1U-NoLED"
 			(at 120.65 88.9 0)
 			(effects
@@
 			)
 		)
-		(property "Footprint" "MX:MXOnly-1U"
+		(property "Footprint" "MX:MXOnly-1U-NoLED"
 			(at 185.42 88.9 0)
 			(effects
@@
 			)
 		)
-		(property "Footprint" "MX:MXOnly-2U"
+		(property "Footprint" "MX:MXOnly-2U-NoLED"
 			(at 336.55 88.9 0)
 			(effects
@@
 			)
 		)
-		(property "Footprint" "MX:MXOnly-1U"
+		(property "Footprint" "MX:MXOnly-1U-NoLED"
 			(at 207.01 139.7 0)
 			(effects
@@
 			)
 		)
-		(property "Footprint" "MX:MXOnly-1U"
+		(property "Footprint" "MX:MXOnly-1U-NoLED"
 			(at 358.14 165.1 0)
 			(effects
@@
 			)
 		)
-		(property "Footprint" "MX:MXOnly-1.25U"
+		(property "Footprint" "MX:MXOnly-1.25U-NoLED"
 			(at 271.78 190.5 0)
 			(effects
@@
 			)
 		)
-		(property "Footprint" "MX:MXOnly-1U"
+		(property "Footprint" "MX:MXOnly-1U-NoLED"
 			(at 77.47 165.1 0)
 			(effects
@@
 			)
 		)
-		(property "Footprint" "MX:MXOnly-1U"
+		(property "Footprint" "MX:MXOnly-1U-NoLED"
 			(at 163.83 165.1 0)
 			(effects
@@
 			)
 		)
-		(property "Footprint" "MX:MXOnly-1U"
+		(property "Footprint" "MX:MXOnly-1U-NoLED"
 			(at 99.06 165.1 0)
 			(effects
@@
 			)
 		)
-		(property "Footprint" "MX:MXOnly-1U"
+		(property "Footprint" "MX:MXOnly-1U-NoLED"
 			(at 358.14 190.5 0)
 			(effects
@@
 			)
 		)
-		(property "Footprint" "MX:MXOnly-1.5U"
+		(property "Footprint" "MX:MXOnly-1.5U-NoLED"
 			(at 55.88 114.3 0)
 			(effects
@@
 			)
 		)
-		(property "Footprint" "MX:MXOnly-1U"
+		(property "Footprint" "MX:MXOnly-1U-NoLED"
 			(at 163.83 139.7 0)
 			(effects
@@
 			)
 		)
-		(property "Footprint" "MX:MXOnly-1U"
+		(property "Footprint" "MX:MXOnly-1U-NoLED"
 			(at 77.47 88.9 0)
 			(effects
@@
 			)
 		)
-		(property "Footprint" "MX:MXOnly-1U"
+		(property "Footprint" "MX:MXOnly-1U-NoLED"
 			(at 293.37 114.3 0)
 			(effects
@@
 			)
 		)
-		(property "Footprint" "MX:MXOnly-1.75U"
+		(property "Footprint" "MX:MXOnly-1.75U-NoLED"
 			(at 314.96 165.1 0)
 			(effects
@@
 			)
 		)
-		(property "Footprint" "MX:MXOnly-1U"
+		(property "Footprint" "MX:MXOnly-1U-NoLED"
 			(at 207.01 165.1 0)
 			(effects
@@
 			)
 		)
-		(property "Footprint" "MX:MXOnly-1.25U"
+		(property "Footprint" "MX:MXOnly-1.25U-NoLED"
 			(at 77.47 190.5 0)
 			(effects
@@
 			)
 		)
-		(property "Footprint" "MX:MXOnly-1.25U"
+		(property "Footprint" "MX:MXOnly-1.25U-NoLED"
 			(at 293.37 190.5 0)
 			(effects
@@
 			)
 		)
-		(property "Footprint" "MX:MXOnly-1U"
+		(property "Footprint" "MX:MXOnly-1U-NoLED"
 			(at 228.6 88.9 0)
 			(effects
@@
 			)
 		)
-		(property "Footprint" "MX:MXOnly-1U"
+		(property "Footprint" "MX:MXOnly-1U-NoLED"
 			(at 336.55 190.5 0)
 			(effects
