File: keyboard/keyboard.kicad_pcb (KiCad board)
At the start: 2 copper layers, 155 parts, among them J1 AVR-ISP-6, SW10 8, SW11 9, SW12 0, SW13 -_, SW14 +=, SW15 BSPC, SW16 DEL, SW17 TAB, SW18 Q, SW19 W, SW2 ESC, SW20 E, SW21 R, SW22 T, SW23 Y, SW24 U, SW25 I, SW26 O, SW27 P, SW28 {[, SW29 }], SW3 1, SW30 |\, SW31 PGUP, SW32 CAPS, SW33 A, SW34 S, SW35 D, SW36 F, SW37 G, SW38 H, SW39 J, SW4 2, SW40 K, SW41 L, SW42 :;, SW43 "', SW44 ENTER, SW45 PGDN, SW46 SHIFT, SW47 Z, SW48 X, SW49 C, SW5 3, SW50 V, SW51 B, SW52 N, SW53 M, SW54 <,, SW55 >., SW56 ?/, SW57 SHIFT, SW58 UP, SW59 END, SW6 4, SW60 CTRL, SW61 WIN, SW62 ALT, SW63 SPACE, SW64 FN, SW65 CTRL, SW66 LEFT, SW67 DOWN, SW68 RIGHT, SW7 5, SW8 6, SW9 7, U1 ATmega32U4-A, U2 PRTR5V0U2X, Y1 Crystal_GND24_Small

Commit message: Finished diode layout and changed switch footprints to no-LED
Parts:
- SW1, SW10, SW11, SW12, SW13, SW14, SW16, SW18, SW19, SW2, SW20, SW21, SW22, SW23, SW24, SW25, SW26, SW27, SW28, SW29, SW3, SW31, SW33, SW34, SW35, SW36, SW37, SW38, SW39, SW4, SW40, SW41, SW42, SW43, SW45, SW47, SW48, SW49, SW5, SW50, SW51, SW52, SW53, SW54, SW55, SW56, SW58, SW59, SW6, SW66, SW67, SW68, SW7, SW8, SW9: footprint MX:MXOnly-1U -> MX:MXOnly-1U-NoLED
- SW15: footprint MX:MXOnly-2U -> MX:MXOnly-2U-NoLED
- SW17, SW30, SW60, SW62: footprint MX:MXOnly-1.5U -> MX:MXOnly-1.5U-NoLED
- SW32, SW57: footprint MX:MXOnly-1.75U -> MX:MXOnly-1.75U-NoLED
- SW44, SW46: footprint MX:MXOnly-2.25U -> MX:MXOnly-2.25U-NoLED
- SW61, SW64, SW65: footprint MX:MXOnly-1.25U -> MX:MXOnly-1.25U-NoLED
- SW63: footprint MX:MXOnly-6.25U -> MX:MXOnly-6.25U-ReversedStabilizers-NoLED
- moved D1 293.6 mm to (15.9, -89.7), turned to -90 degrees
- moved D16 279.9 mm to (20.6, -70.6), turned to -90 degrees
- moved D2 279.4 mm to (34.9, -89.7), turned to -90 degrees
- moved D31 268.2 mm to (23.0, -51.6), turned to -90 degrees
- moved D3 266.0 mm to (54.0, -89.7), turned to -90 degrees
- moved D17 261.7 mm to (44.5, -70.6), turned to -90 degrees
- moved D4 253.2 mm to (73.0, -89.7), turned to -90 degrees
- moved D45 252.9 mm to (27.8, -32.5), turned to -90 degrees
- moved D18 248.3 mm to (63.5, -70.6), turned to -90 degrees
- moved D59 248.3 mm to (20.6, -13.5), turned to -90 degrees
- moved D32 247.9 mm to (49.2, -51.6), turned to -90 degrees
- moved D5 241.4 mm to (92.1, -89.7), turned to -90 degrees
- moved D19 235.8 mm to (82.5, -70.6), turned to -90 degrees
- moved D33 234.5 mm to (68.3, -51.6), turned to -90 degrees
- moved D6 230.6 mm to (111.1, -89.7), turned to -90 degrees
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
Commit message: Crudely arranged USB-C and MCU footprints and cut PCB edges.
Parts:
- SW1: footprint MX:MXOnly-1U-NoLED -> Button_Switch_SMD:SW_SPST_SKQG_WithStem
- moved USB1 259.4 mm to (152.4, -110.3), turned to 0 degrees
- moved R5 254.7 mm to (141.1, -101.6)
- moved U2 250.4 mm to (152.4, -96.0), turned to 0 degrees
- moved R6 248.8 mm to (160.1, -101.6), turned to 0 degrees
- moved F1 241.4 mm to (155.6, -89.0), turned to -90 degrees
- moved C8 194.4 mm to (157.2, -28.6), turned to -90 degrees
- moved C6 189.2 mm to (151.6, -24.1), turned to 90 degrees
- moved J1 188.3 mm to (108.4, -18.9)
- moved C7 185.0 mm to (151.6, -15.6), turned to -90 degrees
- moved R3 184.0 mm to (158.8, -35.5), turned to -90 degrees
- moved R4 183.3 mm to (162.7, -34.3), turned to -90 degrees
- moved C1 174.0 mm to (163.5, -29.1), turned to -90 degrees
- moved SW1 172.3 mm to (182.6, -27.0)
- moved C4 170.5 mm to (171.4, -21.4)
- moved R2 166.8 mm to (172.2, -26.8), turned to 90 degrees
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Connections:
- R6 pad 1: VCC -> Net-(USB1-CC2)
- USB1 pad 10: VCC -> Net-(USB1-CC2)
Other:
- board outline added: 304.8 x 99.2 mm
